File: Sony_keyboard/Sony_keyboard.brd (EAGLE design)
At the start: 63.2 x 36.8 mm, 7 parts, among them J1 3pin, J10 20pin, J2 5pin, U1 FPC24, U2 Teensy++2.0

Commit message: Add files via upload
Parts:
- added U$1: (no value), oshw:OSHW_5MM
Changed lines of the file:
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@@
 <?xml version="1.0" encoding="utf-8"?>
 <!DOCTYPE eagle SYSTEM "eagle.dtd">
-<eagle version="8.2.2">
+<eagle version="9.2.2">
 <drawing>
 <settings>
-<setting alwaysvectorfont="no"/>
+<setting alwaysvectorfont="yes"/>
+<setting keepoldvectorfont="yes"/>
 <setting verticaltext="up"/>
 </settings>
@@
 <param name="dpMaxLengthDifference" value="10mm"/>
 <param name="dpGapFactor" value="2.5"/>
-<param name="checkGrid" value="0"/>
 <param name="checkAngle" value="0"/>
 <param name="checkFont" value="1"/>
 <param name="checkRestrict" value="1"/>
+<param name="checkStop" value="0"/>
+<param name="checkValues" value="0"/>
+<param name="checkNames" value="1"/>
+<param name="checkWireStubs" value="1"/>
+<param name="checkPolygonWidth" value="0"/>
 <param name="useDiameter" value="13"/>
 <param name="maxErrors" value="50"/>
@@
 </autorouter>
 <elements>
-<element name="C1" library="SparkFun-Capacitors" package="0603" value="10uF" x="8.89" y="5.08">
+<element name="C1" library="SparkFun-Capacitors" package="0603" value="10uF" x="8.89" y="5.08" smashed="yes">
+<attribute name="NAME" x="8.89" y="5.842" size="0.6096" layer="25" font="vector" ratio="20" align="bottom-center"/>
 <attribute name="PROD_ID" value="CAP-11015" x="8.89" y="5.08" size="1.778" layer="27" display="off"/>
+<attribute name="VALUE" x="8.89" y="4.318" size="0.6096" layer="27" font="vector" ratio="20" align="top-center"/>
 </element>
-<element name="C2" library="SparkFun-Capacitors" package="0603" value="1.0uF" x="8.89" y="2.54">
+<element name="C2" library="SparkFun-Capacitors" package="0603" value="1.0uF" x="8.89" y="2.54" smashed="yes">
+<attribute name="NAME" x="8.89" y="3.302" size="0.6096" layer="25" font="vector" ratio="20" align="bottom-center"/>
 <attribute name="PROD_ID" value="CAP-00868" x="8.89" y="2.54" size="1.778" layer="27" display="off"/>
+<attribute name="VALUE" x="8.89" y="1.778" size="0.6096" layer="27" font="vector" ratio="20" align="top-center"/>
 </element>
-<element name="J1" library="SparkFun-Connectors" package="1X03" value="3pin" x="60.96" y="19.05" rot="R90"/>
-<element name="J10" library="SparkFun-Connectors" package="1X20" value="20pin" x="7.62" y="34.29"/>
-<element name="J2" library="SparkFun-Connectors" package="1X05" value="5pin" x="7.62" y="8.89"/>
-<element name="U1" library="FPC CONN" package="FPC24" value="FPC24" x="41.91" y="2.54" rot="R180"/>
-<element name="U2" library="Teensy" package="TEENSYPP2.0" value="Teensy++2.0" x="31.75" y="21.59"/>
+<element name="J1" library="SparkFun-Connectors" package="1X03" value="3pin" x="60.96" y="19.05" smashed="yes" rot="R90">
+<attribute name="NAME" x="59.563" y="17.78" size="0.6096" layer="25" font="vector" ratio="20" rot="R90"/>
+<attribute name="VALUE" x="62.992" y="17.78" size="0.6096" layer="27" font="vector" ratio="20" rot="R90"/>
+</element>
+<element name="J10" library="SparkFun-Connectors" package="1X20" value="20pin" x="7.62" y="34.29" smashed="yes">
+<attribute name="NAME" x="6.35" y="35.687" size="0.6096" layer="25" font="vector" ratio="20"/>
+<attribute name="VALUE" x="6.35" y="32.258" size="0.6096" layer="27" font="vector" ratio="20"/>
+</element>
+<element name="J2" library="SparkFun-Connectors" package="1X05" value="5pin" x="7.62" y="8.89" smashed="yes">
+<attribute name="NAME" x="6.35" y="10.287" size="0.6096" layer="25" font="vector" ratio="20"/>
+<attribute name="VALUE" x="6.35" y="6.858" size="0.6096" layer="27" font="vector" ratio="20"/>
+</element>
+<element name="U1" library="FPC CONN" package="FPC24" value="FPC24" x="41.91" y="2.54" smashed="yes" rot="R180"/>
+<element name="U2" library="Teensy" package="TEENSYPP2.0" value="Teensy++2.0" x="31.75" y="21.59" smashed="yes"/>
+<element name="U$1" library="oshw" package="OSHW_5MM" value="" x="21.59" y="5.08" smashed="yes"/>
 </elements>
 <signals>
@@
 </signal>
 </signals>
+<mfgpreviewcolors>
+<mfgpreviewcolor name="soldermaskcolor" color="0xC8008000"/>
+<mfgpreviewcolor name="silkscreencolor" color="0xFFFEFEFE"/>
+<mfgpreviewcolor name="backgroundcolor" color="0xFF282828"/>
+<mfgpreviewcolor name="coppercolor" color="0xFFFFBF00"/>
+<mfgpreviewcolor name="substratecolor" color="0xFF786E46"/>
+</mfgpreviewcolors>
 </board>
 </drawing>
+<compatibility>
+<note version="6.3" minversion="6.2.2" severity="warning">
+Since Version 6.2.2 text objects can contain more than one line,
+which will not be processed correctly with this version.
+</note>
+</compatibility>
 </eagle>
